Commit message: Sun Mar 10 01:30:04 CST 2019 add the second laser and tuning the original laser model parameters

File: robots/youbot.urdf.xacro (robot description, xacro)
@@ -42,6 +42,10 @@
   </xacro:youbot_gripper>
   <!-- base laser front -->
-  <xacro:hokuyo_urg04_laser name="base_laser_front" parent="base" ros_topic="scan_front" update_rate="10" min_angle="-1.57" max_angle="1.57">
+  <xacro:hokuyo_urg04_laser name="base_laser_front" parent="base" ros_topic="scan_front" update_rate="40" min_angle="-1.57" max_angle="1.57">
     <origin xyz="0.3 0 -0.03" rpy="0 0 0"/>
   </xacro:hokuyo_urg04_laser>
+  <!-- base laser back -->
+  <xacro:hokuyo_urg04_laser name="base_laser_back" parent="base" ros_topic="scan_back" update_rate="40" min_angle="-1.57" max_angle="1.57">
+    <origin xyz="-0.3 0 -0.03" rpy="0 0 3.14"/>
+  </xacro:hokuyo_urg04_laser>
 </robot>

File: urdf/sensors/hokuyo_urg04_laser.gazebo.xacro (robot description, xacro)
@@ -7,22 +7,22 @@
     <gazebo reference="${name}_link">
       <sensor name="${name}" type="ray">
-		<always_on>true</always_on>
+    		<always_on>true</always_on>
         <update_rate>${update_rate}</update_rate>
-		<pose>0 0 0 0 0 0</pose>
-		<visualize>false</visualize>
+    		<pose>0 0 0 0 0 0</pose>
+    		<visualize>false</visualize>
         <ray>
-            <scan>
+         <scan>
                 <horizontal>
-                    <samples>150</samples>
+                    <samples>720</samples>
                     <resolution>1.0</resolution>
                     <min_angle>${min_angle}</min_angle>
                     <max_angle>${max_angle}</max_angle>
                 </horizontal>
-            </scan>
-            <range>
-				<min>0.05</min>
-				<max>5.6</max>
-				<resolution>0.36</resolution>
-			</range>
+         </scan>
+         <range>
+				       <min>0.05</min>
+				       <max>5.6</max>
+				       <resolution>0.01</resolution>
+			   </range>
         </ray>
         <plugin name="gazebo_ros_${name}_controller" filename="libgazebo_ros_laser.so">

Commit message: Mon Mar 11 01:48:01 CST 2019add intel d435 to youbot.urdf.xacro

File: robots/youbot.urdf.xacro (robot description, xacro)
@@ -22,4 +22,5 @@
   <!-- sensors -->
   <xacro:include filename="$(find youbot_description)/urdf/sensors/hokuyo_urg04_laser.urdf.xacro"/>
+  <xacro:include filename="$(find youbot_description)/urdf/sensors/_d435.urdf.xacro"/>
   <!-- Now we can start using the macros xacro:included above to define the actual youbot -->
   <!-- The first use of a macro.  This one was defined in base.urdf.xacro above.
@@ -49,3 +50,6 @@
     <origin xyz="-0.3 0 -0.03" rpy="0 0 3.14"/>
   </xacro:hokuyo_urg04_laser>
+  <xacro:sensor_d435 parent="base_link">
+    <origin xyz="0.3 0 0.03" rpy="0 0 0"/>
+  </xacro:sensor_d435>
 </robot>
